File: hardware/ovc4/carrier/interfaces.sch (KiCad schematic (older format))
At the start: 9 parts, among them Q3 NMOS, U1 Jetson_Nano, U16 TCA9803

Commit message: Several camera interface + USB fixes
Signed-off-by: Luca Della Vedova <luca@openrobotics.org>
Parts:
- added C? (x6): 100n, Capacitor_SMD:C_0402_1005Metric, symbol Device:C_Small
- added R? (x2): 110R, Resistor_SMD:R_0402_1005Metric, symbol Device:R_Small
- added R? (x4): 2k2, Resistor_SMD:R_0402_1005Metric, symbol Device:R_Small
- added U?: ARJ11C-MBSAS-A-BA-7MU2, Ethernet:ARJ11C-MBSAS-A-BA-7MU2, symbol ethernet:ARJ11C-MBSAS-A-BA-7MU2
- added U? (x2): TCA9803, Package_SO:VSSOP-8_3.0x3.0mm_P0.65mm, symbol Interface:TCA9803
- Q3: value NMOS -> DMN65D8L; footprint (none) -> Package_TO_SOT_SMD:SOT-23; symbol Device:Q_NMOS_GDS -> Device:Q_NMOS_GSD
Connections:
- net labels added: CAM0_SCL_1V8, CAM0_SCL_3V3, CAM0_SDA_1V8, CAM0_SDA_3V3, CAM1_SCL_1V8, CAM1_SCL_3V3, CAM1_SDA_1V8, CAM1_SDA_3V3, FRAME_TRIGGER, GBE_LED_ACT, GBE_LED_LINK, GBE_MDI0_N, GBE_MDI0_P, GBE_MDI1_N, GBE_MDI1_P, GBE_MDI2_N, GBE_MDI2_P, GBE_MDI3_N, GBE_MDI3_P, NX_MCU_BOOT, NX_MCU_nRST, PICAM0_SCL_1V8, PICAM0_SCL_3V3, PICAM0_SDA_1V8, PICAM0_SDA_3V3, PICAM1_SCL_1V8, PICAM1_SDA_1V8, VBUS
- net labels removed: CAM0_SCL, CAM0_SDA, CAM1_SCL, CAM1_SDA, NX_MCU_GPIO1, NX_MCU_GPIO2, PICAM1_SCL, PICAM1_SDA, USB0_VBUS_5V
- wire segments 33 -> 76
Other:
- note added: "I2C0 ,I2C1 and CAM_I2C are 3.3V\nI2C2 is 1.8V"
- note added: "It seems the CAM_I2C interface\nhas pullups on Jetson module"
- note added: "USB chip as VIH of 1.2V\nPIcam has a FET used as a shifter"
- note removed: "I2C0 and 1 are 3.3V\nI2C2 is 1.8V\nI2C2 shifted (check if necessary)"
- moved on the sheet: R32, R33
