File: hardware/ovc4/carrier/usb.sch (KiCad schematic (older format))
At the start: 52 parts, among them J1 USB_B_Micro, J2 USB_C_Receptacle, Q1 SI2369DS, Q2 SI2369DS, U1 Jetson_Nano, U2 STUSB4500, U3 CY7C65642-28LTXC, U4 HD3SS3202, U5 LM3526-L, Y1 12MHz

Commit message: Several camera interface + USB fixes
Signed-off-by: Luca Della Vedova <luca@openrobotics.org>
Parts:
- removed J1: USB_B_Micro, Connector_USB:USB_Micro-B_Wuerth_629105150521_CircularHoles, symbol Connector:USB_B_Micro
- removed R14: 10k, Resistor_SMD:R_0402_1005Metric, symbol Device:R_Small
- added C? (x2): 100n, Capacitor_SMD:C_0402_1005Metric, symbol Device:C_Small
- added C? (x2): 120u, Capacitor_SMD:C_1206_3216Metric, symbol Device:C_Small
- added D? (x2): D_TVS_x2_AAC, USB:TPD2EUSB30x, symbol Device:D_TVS_x2_AAC
- added L? (x4): 220, Inductor_SMD:L_0603_1608Metric, symbol Device:L_Small
- added U?: USBA_DUAL, USB:USBA_DUAL_HOR, symbol usb2_connector:USBA_DUAL
Connections:
- net labels added: GBE_LED_ACT, GBE_LED_LINK, GBE_MDI0_N, GBE_MDI0_P, GBE_MDI1_N, GBE_MDI1_P, GBE_MDI2_N, GBE_MDI2_P, GBE_MDI3_N, GBE_MDI3_P, VBUS_USER0, VBUS_USER1
- net labels removed: HUB_nOVR4, USB0_VBUS_5V, USB1_D_N, USB1_D_P
- wire segments 194 -> 208
- no-connect marks 14 -> 16
Other:
- note added: "USB0 is the only USB with a VBUS detect line (for device mode)\nTODO dev guide suggests using USB2?"
- note removed: "MCU HS USB"
- note removed: "Pullups in level translator"
- note removed: "TODO ESD protection on external USB ports"
- note removed: "TODO add user USB ports"
- note removed: "TODO check that 3V3 unavailable on powerup is OK"
- moved on the sheet: C20, C22, R15, R16, R17, U5
